Commit message: 接入 go2_1 在线视觉感知并重构动态追踪控制（单狗稳定跟随）
- 目标源可切到 go2_1 在线感知估计：新增 target_perception / perception_eval
- 相机 xacro 升级为 RGB-D；dynamic_encircle 增加丢目标 coast/外推兜底
- formation 重构为“锁定行人的定距跟随”，解决反复切换/S弯/近处大转向丢视野
- 新增一键脚本 start_three_go2_dynamic_tracking.sh（当前仅启用 go2_1）
- 同步更新 README / 修改记录汇总 / 情况说明；YOLO 权重 *.pt 加入 .gitignore

Co-Authored-By: Claude Opus 4.8 <noreply@anthropic.com>

File: go2_ws_v2/src/unitree-go2-ros2/robots/descriptions/go2_description/xacro/camera_rgb_3d.xacro (robot description, xacro)
@@ -1,5 +1,5 @@
 <?xml version="1.0"?>
-<!-- Lightweight RGB-only camera for the multi-dog 3D chain. Each dog must
-     publish its own image on /go2_i/camera/image_raw with no cross-talk.
+<!-- RGB-D depth camera for the multi-dog 3D chain. Each dog must publish its
+     own RGB + depth on /go2_i/camera/... with no cross-talk.
      IMPORTANT multi-dog gotcha (verified live with three dogs in one gzserver)
      gazebo_ros_camera does NOT honor an absolute remapping the way the velodyne
@@ -14,4 +14,8 @@
      to /go2_i/camera/image_raw. frame_name still uses frame_prefix and is read
      correctly per dog. Low resolution and visualize=false to keep GPU cost down.
+     This is a type=depth sensor so the single plugin publishes both the RGB
+     stream (/go2_i/camera/image_raw + /go2_i/camera/camera_info) and the depth
+     stream (/go2_i/camera/depth/image_raw 32FC1 in meters
+     + /go2_i/camera/depth/camera_info) plus /go2_i/camera/points.
      NOTE keep comments free of colon-space because robot_description is
      YAML-parsed by launch and a colon-space anywhere breaks it. -->
@@ -40,5 +44,5 @@
     </link>
     <joint name="camera_rgb_joint" type="fixed">
-        <origin rpy="0 0 0" xyz="0.02 0 0"/>
+        <origin rpy="0 0 0" xyz="0.02 -0.02 0"/>
         <parent link="camera_link"/>
         <child link="camera_rgb_frame"/>
@@ -51,19 +55,31 @@
     </joint>
     <link name="camera_rgb_optical_frame"/>
-    <gazebo reference="camera_rgb_frame">
-        <sensor name="camera_rgb" type="camera">
+    <joint name="camera_depth_joint" type="fixed">
+        <origin rpy="0 0 0" xyz="0.02 0.02 0"/>
+        <parent link="camera_link"/>
+        <child link="camera_depth_frame"/>
+    </joint>
+    <link name="camera_depth_frame"/>
+    <joint name="camera_depth_optical_joint" type="fixed">
+        <origin rpy="-1.5707963267948966 0 -1.5707963267948966" xyz="0 0 0"/>
+        <parent link="camera_depth_frame"/>
+        <child link="camera_depth_optical_frame"/>
+    </joint>
+    <link name="camera_depth_optical_frame"/>
+    <gazebo reference="camera_depth_frame">
+        <sensor name="camera_rgbd" type="depth">
             <always_on>true</always_on>
             <visualize>false</visualize>
-            <update_rate>10</update_rate>
+            <update_rate>15</update_rate>
             <camera name="camera">
                 <horizontal_fov>1.047</horizontal_fov>
                 <image>
-                    <width>320</width>
-                    <height>240</height>
+                    <width>640</width>
+                    <height>480</height>
                     <format>R8G8B8</format>
                 </image>
                 <clip>
                     <near>0.05</near>
-                    <far>100.0</far>
+                    <far>50.0</far>
                 </clip>
             </camera>
@@ -73,5 +89,8 @@
                 </ros>
                 <camera_name>$(arg robot_namespace)/camera</camera_name>
-                <frame_name>$(arg frame_prefix)camera_rgb_optical_frame</frame_name>
+                <frame_name>$(arg frame_prefix)camera_depth_optical_frame</frame_name>
+                <hack_baseline>0.04</hack_baseline>
+                <min_depth>0.05</min_depth>
+                <max_depth>25.0</max_depth>
             </plugin>
         </sensor>
